File: Protomatrix/Protomatrix.kicad_pcb (KiCad board)
At the start: 2 copper layers, 140 parts, among them J1 Conn_01x21_Female

Commit message: more updates
Parts:
- removed MXE1, MXQ1, MXR1, MXT1, MXU1, MXW1, MXY1: MX-NoLED, MX_Only:MXOnly-1U-NoLED
- added MX-E1: MX-NoLED, MX_Only:MXOnly-1U-NoLED, F.Cu at (-65.1, 92.1)
- added MX-Q1: MX-NoLED, MX_Only:MXOnly-1U-NoLED, F.Cu at (-103.2, 92.1)
- added MX-R1: MX-NoLED, MX_Only:MXOnly-1U-NoLED, F.Cu at (-46.0, 92.1)
- added MX-T1: MX-NoLED, MX_Only:MXOnly-1U-NoLED, F.Cu at (-27.0, 92.1)
- added MX-U1: MX-NoLED, MX_Only:MXOnly-1U-NoLED, F.Cu at (11.1, 92.1)
- added MX-W1: MX-NoLED, MX_Only:MXOnly-1U-NoLED, F.Cu at (-84.1, 92.1)
- added MX-Y1: MX-NoLED, MX_Only:MXOnly-1U-NoLED, F.Cu at (-7.94, 92.1)
- added MX-\1: MX-NoLED, MX_Only:MXOnly-1.5U-NoLED, F.Cu at (130.2, 92.1)
- moved MX-,1 514.2 mm to (44.5, 130.2)
- moved MX-[1 444.9 mm to (87.3, 92.1)
- moved MX-]1 338.9 mm to (106.4, 92.1)
- moved MX-l1 325.2 mm to (54.0, 111.1)
- moved D33 239.6 mm to (-30.2, -3.97)
- moved D32 239.5 mm to (-36.5, -3.97)
- moved MX-Enter1 234.6 mm to (123.0, 111.1)
- moved MX-Right1 233.4 mm to (160.3, 149.2)
- moved D34 226.1 mm to (-131.0, -3.97), turned to 270 degrees
- moved MX-Del1 196.9 mm to (158.8, 92.1)
- moved MX-Ins1 196.9 mm to (158.8, 73.0)
- moved MX-PgDn1 196.9 mm to (196.8, 92.1)
- moved MX-PgUp1 196.9 mm to (196.8, 73.0)
- moved MX-Hm1 196.9 mm to (177.8, 73.0)
- moved MX-end1 196.9 mm to (177.8, 92.1)
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Connections:
- D34 pad 1: Net-(D34-Pad1) -> Row1
- D64 pad 2: Row3 -> Net-(D64-Pad2)
- MX-Spc1 pad 2: Row3 -> Net-(D64-Pad2)

Commit message: routing & more
Parts:
- J1: value Conn_01x21_Female -> Conn_01x18_Female; footprint Connector_PinHeader_2.54mm:PinHeader_1x21_P2.54mm_Horizontal -> Connector_PinHeader_2.54mm:PinHeader_1x18_P2.54mm_Vertical
- moved D35 219.9 mm to (-129.6, 39.9), turned to 180 degrees
- moved D48 217.8 mm to (-129.6, 46.3), turned to 180 degrees
- moved D61 216.1 mm to (-129.6, 53.4), turned to 180 degrees
- moved D36 213.6 mm to (-116.6, 39.9), turned to 180 degrees
- moved D49 211.4 mm to (-116.6, 46.3), turned to 180 degrees
- moved D62 210.1 mm to (-116.9, 53.4), turned to 180 degrees
- moved D37 207.4 mm to (-103.5, 39.9), turned to 180 degrees
- moved D50 205.1 mm to (-103.6, 46.3), turned to 180 degrees
- moved D63 203.4 mm to (-103.4, 53.4), turned to 180 degrees
- moved D38 201.2 mm to (-90.5, 39.9), turned to 180 degrees
- moved D51 198.8 mm to (-90.5, 46.3), turned to 180 degrees
- moved D39 195.0 mm to (-77.5, 39.9), turned to 180 degrees
- moved D52 192.6 mm to (-77.5, 46.3), turned to 180 degrees
- moved D40 188.9 mm to (-64.4, 39.9), turned to 180 degrees
- moved D53 186.4 mm to (-64.5, 46.3), turned to 180 degrees
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- renumbered MX-Lshift1 to MX-LShift1
Connections:
- D15 pad 1: Row0 -> Row2
- D16 pad 1: Row0 -> Row4
- D17 pad 1: Row0 -> Row4
- D31 pad 1: Row1 -> Row3
- D32 pad 1: Row1 -> Row4
- D33 pad 1: Row1 -> Row4
- MX-Del1 pad 1: Col14 -> Col13
- MX-Down1 pad 1: Col15 -> Col8
- MX-Hm1 pad 1: Col15 -> Col13
- MX-Ins1 pad 1: Col14 -> Col13
- MX-LShift1 pad 1: Col12 -> Col0
- MX-LShift1 pad 2: Net-(D59-Pad2) -> Net-(D48-Pad2)
- MX-Left1 pad 1: Col14 -> Col7
- MX-PgDn1 pad 1: Col16 -> Col10
- MX-PgUp1 pad 1: Col16 -> Col11
- MX-RAlt1 pad 1: Col10 -> Col4
- MX-RCtrl1 pad 1: Col12 -> Col6
- MX-RShift1 pad 1: Col0 -> Col11
- MX-RShift1 pad 2: Net-(D48-Pad2) -> Net-(D59-Pad2)
- MX-RSys1 pad 1: Col11 -> Col5
- MX-Right1 pad 1: Col16 -> Col9
- MX-Spc1 pad 1: Col5 -> Col3
- MX-Up1 pad 1: Col15 -> Net-(MX-Up1-Pad1)
- MX-end1 pad 1: Col15 -> Net-(MX-Up1-Pad1)
Routing:
- net Net-(D63-Pad2): track 0.00 -> 142.9 mm
- net Net-(D62-Pad2): track 0.00 -> 141.6 mm
- net Net-(D51-Pad2): track 0.00 -> 119.4 mm
- net Net-(D50-Pad2): track 0.00 -> 113.0 mm
- net Net-(D61-Pad2): track 0.00 -> 112.2 mm
- net Net-(D49-Pad2): track 0.00 -> 107.3 mm
- net Net-(D38-Pad2): track 0.00 -> 102.1 mm
- net Net-(D37-Pad2): track 0.00 -> 95.5 mm
- net Net-(D48-Pad2): track 0.00 -> 95.0 mm
- net Net-(D21-Pad2): track 0.00 -> 91.8 mm
- net Net-(D39-Pad2): track 0.00 -> 90.2 mm
- net Net-(D36-Pad2): track 0.00 -> 89.4 mm
- net Net-(D20-Pad2): track 0.00 -> 85.3 mm
- net Net-(D35-Pad2): track 0.00 -> 81.0 mm
- net Net-(D19-Pad2): track 0.00 -> 78.8 mm
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Other:
- board outline added: 359.6 x 142.1 mm
- net class Default: trace_width 0.25 -> 0.254
- net class Power added: clearance 0.2, trace_width 0.381, via_dia 0.8, via_drill 0.4

Commit message: yep
Routing:
- net Net-(D52-Pad2): track 0.00 -> 125.9 mm
- net Net-(D6-Pad2): track 0.00 -> 41.3 mm
- net Net-(D39-Pad2): track 90.2 -> 108.6 mm
Changed lines of the file:
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@@
     (thickness 1.6)
     (drawings 12)
-    (tracks 275)
+    (tracks 300)
     (zones 0)
     (modules 141)
@@
   (segment (start -83.38501 61.64899) (end -69.534943 61.648991) (width 0.254) (layer F.Cu) (net 6))
   (segment (start -89.154 55.88) (end -83.38501 61.64899) (width 0.254) (layer F.Cu) (net 6))
+  (segment (start -72.01297 27.78125) (end -76.10872 31.877) (width 0.254) (layer F.Cu) (net 7))
+  (segment (start -76.10872 31.877) (end -76.10872 55.71728) (width 0.254) (layer F.Cu) (net 7))
+  (segment (start -76.10872 55.71728) (end -72.009 59.817) (width 0.254) (layer F.Cu) (net 7))
+  (segment (start -72.009 59.817) (end -68.79867 59.817) (width 0.254) (layer F.Cu) (net 7))
+  (segment (start -68.79867 59.817) (end -66.93171 61.68396) (width 0.254) (layer F.Cu) (net 7))
   (segment (start -100.75875 86.995) (end -100.6475 86.995) (width 0.254) (layer F.Cu) (net 19))
   (segment (start -105.545499 82.208251) (end -100.75875 86.995) (width 0.254) (layer F.Cu) (net 19))
@@
   (segment (start -66.72899 82.171444) (end -63.810434 85.09) (width 0.254) (layer F.Cu) (net 41))
   (segment (start -63.810434 85.09) (end -60.071 85.09) (width 0.254) (layer F.Cu) (net 41))
-  (segment (start -85.084584 39.91) (end -88.24598 43.071396) (width 0.254) (layer F.Cu) (net 42))
-  (segment (start -88.24598 43.071396) (end -88.24598 55.503888) (width 0.254) (layer F.Cu) (net 42))
-  (segment (start -88.24598 55.503888) (end -83.008896 60.740972) (width 0.254) (layer F.Cu) (net 42))
-  (segment (start -83.008896 60.740972) (end -69.15883 60.740973) (width 0.254) (layer F.Cu) (net 42))
-  (segment (start -69.15883 60.740973) (end -69.158829 60.740973) (width 0.254) (layer F.Cu) (net 42))
+  (segment (start -38.1 105.41) (end -38.735 106.045) (width 0.254) (layer F.Cu) (net 42))
+  (segment (start -38.1 87.884) (end -38.1 105.41) (width 0.254) (layer F.Cu) (net 42))
   (segment (start -69.158829 60.740973) (end -67.307822 62.59198) (width 0.254) (layer F.Cu) (net 42))
+  (segment (start -88.24598 55.503888) (end -83.008896 60.740972) (width 0.254) (layer F.Cu) (net 42))
   (segment (start -50.557953 62.59198) (end -47.55199 65.597943) (width 0.254) (layer F.Cu) (net 42))
+  (segment (start -85.084584 39.91) (end -88.24598 43.071396) (width 0.254) (layer F.Cu) (net 42))
+  (segment (start -83.008896 60.740972) (end -69.158829 60.740973) (width 0.254) (layer F.Cu) (net 42))
+  (segment (start -40.894 85.09) (end -38.1 87.884) (width 0.254) (layer F.Cu) (net 42))
+  (segment (start -88.24598 43.071396) (end -88.24598 55.503888) (width 0.254) (layer F.Cu) (net 42))
   (segment (start -67.307822 62.59198) (end -50.557953 62.59198) (width 0.254) (layer F.Cu) (net 42))
+  (segment (start -44.704 85.09) (end -40.894 85.09) (width 0.254) (layer F.Cu) (net 42))
   (segment (start -47.55199 65.597943) (end -47.55199 82.24201) (width 0.254) (layer F.Cu) (net 42))
   (segment (start -47.55199 82.24201) (end -44.704 85.09) (width 0.254) (layer F.Cu) (net 42))
-  (segment (start -44.704 85.09) (end -40.894 85.09) (width 0.254) (layer F.Cu) (net 42))
-  (segment (start -40.894 85.09) (end -38.1 87.884) (width 0.254) (layer F.Cu) (net 42))
   (segment (start -115.3 108.1725) (end -115.3 123.095) (width 0.254) (layer F.Cu) (net 51))
   (segment (start -123.55198 65.298886) (end -123.55198 84.197204) (width 0.254) (layer F.Cu) (net 51))
@@
   (segment (start -63.754 84.455) (end -63.754 84.504368) (width 0.254) (layer F.Cu) (net 55))
   (segment (start -63.754 84.504368) (end -63.622378 84.63599) (width 0.254) (layer F.Cu) (net 55))
+  (segment (start -33.02 106.68) (end -33.02 121.92) (width 0.254) (layer F.Cu) (net 56))
+  (segment (start -35.56 104.14) (end -33.02 106.68) (width 0.254) (layer F.Cu) (net 56))
+  (segment (start -37.64599 104.08601) (end -37.592 104.14) (width 0.254) (layer F.Cu) (net 56))
+  (segment (start -82.820839 60.286963) (end -68.970772 60.286964) (width 0.254) (layer F.Cu) (net 56))
+  (segment (start -47.09798 82.053954) (end -44.515944 84.63599) (width 0.254) (layer F.Cu) (net 56))
+  (segment (start -37.64599 87.695943) (end -37.64599 104.08601) (width 0.254) (layer F.Cu) (net 56))
+  (segment (start -87.79197 55.315832) (end -82.820839 60.286963) (width 0.254) (layer F.Cu) (net 56))
+  (segment (start -68.970772 60.286964) (end -67.119766 62.13797) (width 0.254) (layer F.Cu) (net 56))
+  (segment (start -50.369896 62.13797) (end -47.09798 65.409886) (width 0.254) (layer F.Cu) (net 56))
+  (segment (start -85.1375 46.26) (end -87.79197 48.91447) (width 0.254) (layer F.Cu) (net 56))
+  (segment (start -32.004 122.301) (end -29.21 125.095) (width 0.254) (layer F.Cu) (net 56))
+  (segment (start -87.79197 48.91447) (end -87.79197 55.315832) (width 0.254) (layer F.Cu) (net 56))
+  (segment (start -32.639 122.301) (end -32.004 122.301) (width 0.254) (layer F.Cu) (net 56))
+  (segment (start -37.592 104.14) (end -35.56 104.14) (width 0.254) (layer F.Cu) (net 56))
+  (segment (start -67.119766 62.13797) (end -50.369896 62.13797) (width 0.254) (layer F.Cu) (net 56))
+  (segment (start -40.705943 84.63599) (end -37.64599 87.695943) (width 0.254) (layer F.Cu) (net 56))
+  (segment (start -33.02 121.92) (end -32.639 122.301) (width 0.254) (layer F.Cu) (net 56))
+  (segment (start -47.09798 65.409886) (end -47.09798 82.053954) (width 0.254) (layer F.Cu) (net 56))
+  (segment (start -44.515944 84.63599) (end -40.705943 84.63599) (width 0.254) (layer F.Cu) (net 56))
   (segment (start -125.054579 63.15422) (end -131.404582 63.15422) (width 0.254) (layer F.Cu) (net 65))
   (segment (start -112.91875 124.84125) (end -114.845991 122.914009) (width 0.254) (layer F.Cu) (net 65))

Commit message: The Routing Continues
Parts:
- moved MX-p1 0.27 mm to (68.3, 92.1)
Connections:
- MX-Up1 pad 1: Net-(MX-Up1-Pad1) -> Col12
- MX-end1 pad 1: Net-(MX-Up1-Pad1) -> Col12
Routing:
- net Net-(D67-Pad2): track 0.00 -> 198.9 mm
- net Net-(D66-Pad2): track 0.00 -> 192.6 mm
- net Net-(D65-Pad2): track 0.00 -> 182.0 mm
- net Net-(D59-Pad2): track 0.00 -> 179.6 mm
- net Net-(D58-Pad2): track 0.00 -> 160.9 mm
- net Net-(D57-Pad2): track 0.00 -> 154.9 mm
- net Net-(D64-Pad2): track 0.00 -> 153.6 mm
- net Net-(D56-Pad2): track 0.00 -> 148.0 mm
- net Net-(D46-Pad2): track 0.00 -> 147.8 mm
- net Net-(D45-Pad2): track 0.00 -> 142.4 mm
- net Net-(D55-Pad2): track 0.00 -> 142.3 mm
- net Net-(D44-Pad2): track 0.00 -> 137.4 mm
- net Net-(D54-Pad2): track 0.00 -> 135.9 mm
- net Net-(D28-Pad2): track 0.00 -> 131.6 mm
- net Net-(D53-Pad2): track 0.00 -> 131.0 mm
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
Commit message: Version 0.1 Complete
Parts:
- J1: value Conn_01x18_Female -> Conn_01x20_Female; footprint Connector_PinHeader_2.54mm:PinHeader_1x18_P2.54mm_Vertical -> Connector_PinHeader_2.54mm:PinHeader_1x20_P2.54mm_Vertical
- moved MX-Left1 38.2 mm to (160.3, 149.2)
- moved MX-Right1 38.2 mm to (198.5, 149.2)
- moved D60 1.52 mm to (65.7, 44.7)
- moved D68 1.52 mm to (52.2, 51.9)
- moved D69 1.52 mm to (65.7, 51.9)
- moved D70 1.52 mm to (78.4, 51.9)
Connections:
- J1 pad 10: Col5 -> Col3
- J1 pad 11: Col6 -> Col4
- J1 pad 12: Col7 -> Col5
- J1 pad 13: Col8 -> Col6
- J1 pad 14: Col9 -> Col7
- J1 pad 15: Col10 -> Col8
- J1 pad 16: Col11 -> Col9
- J1 pad 17: Col12 -> Col10
- J1 pad 18: Col13 -> Col11
- J1 pad 4: Row4 -> Row3
- J1 pad 5: Col0 -> Row4
- J1 pad 6: Col1 -> Net-(J1-Pad6)
- J1 pad 7: Col2 -> Col0
- J1 pad 8: Col3 -> Col1
- J1 pad 9: Col4 -> Col2
Routing:
- net Col4: track 0.00 -> 433.4 mm
- net Col5: track 0.00 -> 422.5 mm
- net Col6: track 0.00 -> 411.0 mm
- net Col7: track 0.00 -> 407.9 mm
- net Col0: track 0.00 -> 394.8 mm
- net Col3: track 0.00 -> 392.6 mm
- net Col8: track 0.00 -> 387.9 mm
- net Col1: track 0.00 -> 386.8 mm
- net Col9: track 0.00 -> 371.0 mm
- net Row3: track 0.00 -> 365.0 mm
- net Col2: track 0.00 -> 364.0 mm
- net Row4: track 0.00 -> 354.8 mm
- net Row2: track 0.00 -> 333.5 mm
- net Col12: track 0.00 -> 331.6 mm
- net Row1: track 0.00 -> 330.0 mm
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