File: Protomatrix/Protomatrix.sch (KiCad schematic (older format))
At the start: 141 parts, among them J1 Conn_01x21_Female

Commit message: Routing and stuff
Parts:
- MX-'1, MX-,1, MX-.1, MX-/1, MX-1, MX-;1, MX-Del1, MX-Down1, MX-Hm1, MX-Ins1, MX-LSys1, MX-Left1, MX-O1, MX-PgDn1, MX-PgUp1, MX-RSys1, MX-Right1, MX-Up1, MX-[1, MX-]1, MX-a1, MX-b1, MX-c1, MX-d1, MX-end1, MX-f1, MX-g1, MX-h1, MX-i1, MX-j1, MX-k1, MX-l1, MX-m1, MX-n1, MX-p1, MX-s1, MX-v1, MX-x1, MX-z1, MX0, MX1, MX2, MX3, MX4, MX5, MX6, MX7, MX8, MX9, MX=1, MXE1, MXQ1, MXR1, MXT1, MXU1, MXW1, MXY1, MX`1: footprint (none) -> MX_Only:MXOnly-1U-NoLED
- MX-Bksp1: footprint (none) -> MX_Only:MXOnly-2U-NoLED
- MX-Caps1: footprint (none) -> MX_Only:MXOnly-1.75U-NoLED
- MX-Enter1, MX-Lshift1: footprint (none) -> MX_Only:MXOnly-2.25U-NoLED
- MX-LAlt1, MX-LCtrl1, MX-RAlt1, MX-RCtrl1, MX-Tab1, MX-\1: footprint (none) -> MX_Only:MXOnly-1.5U-NoLED
- MX-RShift1: footprint (none) -> MX_Only:MXOnly-2.75U-NoLED
- MX-Spc1: footprint (none) -> MX_Only:MXOnly-7U-ReversedStabilizers-NoLED
Connections:
- net Col10: now also MX-RAlt1.1 (COL)
- net Col11: now also MX-RSys1.1 (COL); no longer MX-Lshift1.1 (COL)
- net Col12: now also MX-Lshift1.1 (COL), MX-RCtrl1.1 (COL); no longer MX-Up1.1 (COL)
- net Col14: now also MX-Left1.1 (COL)
- net Col15: now also MX-Down1.1 (COL), MX-Up1.1 (COL)
- net Col16: now also MX-Right1.1 (COL)
- net Col3: no longer MX-Spc1.1 (COL)
- net Col4: no longer MX-RAlt1.1 (COL)
- net Col5: now also MX-Spc1.1 (COL); no longer MX-RSys1.1 (COL)
- net Col6: no longer MX-RCtrl1.1 (COL)
- net Col7: no longer MX-Left1.1 (COL)
- net Col8: no longer MX-Down1.1 (COL)
- net Col9: no longer MX-Right1.1 (COL)
- net Row3: now also D64.2 (A), MX-Spc1.2 (ROW)
Other:
- moved on the sheet: D59, D60, D64, D65, D66, D67, D68, D69, D70, MX-Down1, MX-Left1, MX-Lshift1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

Commit message: more updates
Parts:
- renumbered MXE1 to MX-E1, MXQ1 to MX-Q1, MXR1 to MX-R1, MXT1 to MX-T1, MXU1 to MX-U1, MXW1 to MX-W1, MXY1 to MX-Y1
Connections:
- net Row1: now also D34.1 (K)
- net Row3: no longer D64.2 (A), MX-Spc1.2 (ROW)
- new net: D64.2 (A), MX-Spc1.2 (ROW)
Other:
- moved on the sheet: D34, MX-Tab1
Changed lines of the file:
@@
 	10250 3150 10150 3150
 $Comp
-L MX_Alps_Hybrid:MX-NoLED MXQ1
+L MX_Alps_Hybrid:MX-NoLED MX-Q1
 U 1 1 5FC603D6
 P 2350 3850
-F 0 "MXQ1" H 2383 4073 60  0000 C CNN
+F 0 "MX-Q1" H 2383 4073 60  0000 C CNN
 F 1 "MX-NoLED" H 2383 3999 20  0000 C CNN
 F 2 "MX_Only:MXOnly-1U-NoLED" H 1725 3825 60  0001 C CNN
@@
 	2300 4000 2200 4000
 $Comp
-L MX_Alps_Hybrid:MX-NoLED MXE1
+L MX_Alps_Hybrid:MX-NoLED MX-E1
 U 1 1 5FC60400
 P 3400 3850
-F 0 "MXE1" H 3433 4073 60  0000 C CNN
+F 0 "MX-E1" H 3433 4073 60  0000 C CNN
 F 1 "MX-NoLED" H 3433 3999 20  0000 C CNN
 F 2 "MX_Only:MXOnly-1U-NoLED" H 2775 3825 60  0001 C CNN
@@
 	3350 4000 3250 4000
 $Comp
-L MX_Alps_Hybrid:MX-NoLED MXW1
+L MX_Alps_Hybrid:MX-NoLED MX-W1
 U 1 1 5FC60415
 P 2850 3850
-F 0 "MXW1" H 2883 4073 60  0000 C CNN
+F 0 "MX-W1" H 2883 4073 60  0000 C CNN
 F 1 "MX-NoLED" H 2883 3999 20  0000 C CNN
 F 2 "MX_Only:MXOnly-1U-NoLED" H 2225 3825 60  0001 C CNN
@@
 	2800 4000 2700 4000
 $Comp
-L MX_Alps_Hybrid:MX-NoLED MXT1
+L MX_Alps_Hybrid:MX-NoLED MX-T1
 U 1 1 5FC6042A
 P 4550 3850
-F 0 "MXT1" H 4583 4073 60  0000 C CNN
+F 0 "MX-T1" H 4583 4073 60  0000 C CNN
 F 1 "MX-NoLED" H 4583 3999 20  0000 C CNN
 F 2 "MX_Only:MXOnly-1U-NoLED" H 3925 3825 60  0001 C CNN
@@
 	4500 4000 4400 4000
 $Comp
-L MX_Alps_Hybrid:MX-NoLED MXR1
+L MX_Alps_Hybrid:MX-NoLED MX-R1
 U 1 1 5FC6043F
 P 4000 3850
-F 0 "MXR1" H 4033 4073 60  0000 C CNN
+F 0 "MX-R1" H 4033 4073 60  0000 C CNN
 F 1 "MX-NoLED" H 4033 3999 20  0000 C CNN
 F 2 "MX_Only:MXOnly-1U-NoLED" H 3375 3825 60  0001 C CNN
@@
 	3950 4000 3850 4000
 $Comp
-L MX_Alps_Hybrid:MX-NoLED MXU1
+L MX_Alps_Hybrid:MX-NoLED MX-U1
 U 1 1 5FC60454
 P 5600 3850
-F 0 "MXU1" H 5633 4073 60  0000 C CNN
+F 0 "MX-U1" H 5633 4073 60  0000 C CNN
 F 1 "MX-NoLED" H 5633 3999 20  0000 C CNN
 F 2 "MX_Only:MXOnly-1U-NoLED" H 4975 3825 60  0001 C CNN
@@
 	5550 4000 5450 4000
 $Comp
-L MX_Alps_Hybrid:MX-NoLED MXY1
+L MX_Alps_Hybrid:MX-NoLED MX-Y1
 U 1 1 5FC60469
 P 5050 3850
-F 0 "MXY1" H 5083 4073 60  0000 C CNN
+F 0 "MX-Y1" H 5083 4073 60  0000 C CNN
 F 1 "MX-NoLED" H 5083 3999 20  0000 C CNN
 F 2 "MX_Only:MXOnly-1U-NoLED" H 4425 3825 60  0001 C CNN
@@
 	1    0    0    -1
 $EndComp
-Connection ~ 2200 4300
-Wire Wire Line
-	1700 4050 1600 4050
+Wire Wire Line
+	1700 4000 1600 4000
 $Comp
 L Diode:1N4148 D34
 U 1 1 5FC603F5
-P 1600 4200
-F 0 "D34" H 1600 4417 50  0000 C CNN
-F 1 "1N4148" H 1600 4326 50  0000 C CNN
-F 2 "Diode_THT:D_DO-35_SOD27_P7.62mm_Horizontal" H 1600 4025 50  0001 C CNN
-F 3 "https://assets.nexperia.com/documents/data-sheet/1N4148_1N4448.pdf" H 1600 4200 50  0001 C CNN
-	1    1600 4200
+P 1600 4150
+F 0 "D34" H 1600 4367 50  0000 C CNN
+F 1 "1N4148" H 1600 4276 50  0000 C CNN
+F 2 "Diode_THT:D_DO-35_SOD27_P7.62mm_Horizontal" H 1600 3975 50  0001 C CNN
+F 3 "https://assets.nexperia.com/documents/data-sheet/1N4148_1N4448.pdf" H 1600 4150 50  0001 C CNN
+	1    1600 4150
 	0    -1   -1   0
 $EndComp
@@
 L MX_Alps_Hybrid:MX-NoLED MX-Tab1
 U 1 1 5FC603EB
-P 1750 3900
-F 0 "MX-Tab1" H 1783 4123 60  0000 C CNN
-F 1 "MX-NoLED" H 1783 4049 20  0000 C CNN
-F 2 "MX_Only:MXOnly-1.5U-NoLED" H 1125 3875 60  0001 C CNN
-F 3 "" H 1125 3875 60  0001 C CNN
-	1    1750 3900
-	1    0    0    -1
-$EndComp
-Wire Wire Line
-	1900 2950 1900 3850
+P 1750 3850
+F 0 "MX-Tab1" H 1783 4073 60  0000 C CNN
+F 1 "MX-NoLED" H 1783 3999 20  0000 C CNN
+F 2 "MX_Only:MXOnly-1.5U-NoLED" H 1125 3825 60  0001 C CNN
+F 3 "" H 1125 3825 60  0001 C CNN
+	1    1750 3850
+	1    0    0    -1
+$EndComp
+Wire Wire Line
+	1900 2950 1900 3800
 Connection ~ 1600 6950
 Wire Wire Line
 	1100 6950 1600 6950
-Connection ~ 1900 3850
-Wire Wire Line
-	1900 3850 1900 4700
-Wire Wire Line
-	1150 4300 2200 4300
 Connection ~ 1600 5200
 Connection ~ 1900 4700
@@
 Connection ~ 6950 6950
 Wire Wire Line
-	4400 6650 4400 6050
-Connection ~ 4400 6650
-Wire Wire Line
 	4400 6050 4400 6000
 Wire Wire Line
@@
 	1900 5550 1900 6450
 Connection ~ 1900 5550
+Connection ~ 1900 3800
+Wire Wire Line
+	1900 3800 1900 4700
+Wire Wire Line
+	2200 4300 1600 4300
+Connection ~ 2200 4300
+Connection ~ 1600 4300
+Wire Wire Line
+	1600 4300 1150 4300
 $EndSCHEMATC

Commit message: routing & more
Parts:
- J1: value Conn_01x21_Female -> Conn_01x18_Female; footprint Connector_PinHeader_2.54mm:PinHeader_1x21_P2.54mm_Horizontal -> Connector_PinHeader_2.54mm:PinHeader_1x18_P2.54mm_Vertical; symbol Connector:Conn_01x21_Female -> Connector:Conn_01x18_Female
- MX-LShift1: renamed from MX-RShift1; footprint MX_Only:MXOnly-2.75U-NoLED -> MX_Only:MXOnly-2.25U-NoLED
- MX-RShift1: renamed from MX-Lshift1; footprint MX_Only:MXOnly-2.25U-NoLED -> MX_Only:MXOnly-2.75U-NoLED
Connections:
- net Col10: now also MX-PgDn1.1 (COL); no longer MX-RAlt1.1 (COL)
- net Col11: now also MX-PgUp1.1 (COL), MX-RShift1.1 (COL); no longer MX-RSys1.1 (COL)
- net Col12: no longer MX-RCtrl1.1 (COL), MX-RShift1.1 (COL)
- net Col13: now also MX-Del1.1 (COL), MX-Hm1.1 (COL), MX-Ins1.1 (COL)
- net Col3: now also MX-Spc1.1 (COL)
- net Col4: now also MX-RAlt1.1 (COL)
- net Col5: now also MX-RSys1.1 (COL); no longer MX-Spc1.1 (COL)
- net Col6: now also MX-RCtrl1.1 (COL)
- net Col7: now also MX-Left1.1 (COL)
- net Col8: now also MX-Down1.1 (COL)
- net Col9: now also MX-Right1.1 (COL)
- net Row0: no longer D15.1 (K), D16.1 (K), D17.1 (K)
- net Row1: no longer D31.1 (K), D32.1 (K), D33.1 (K)
- net Row2: now also D15.1 (K)
- net Row3: now also D31.1 (K)
- net Row4: now also D16.1 (K), D17.1 (K), D32.1 (K), D33.1 (K)
- removed net Col14: J1.19 (Pin_19), MX-Del1.1 (COL), MX-Ins1.1 (COL), MX-Left1.1 (COL)
- removed net Col15: J1.20 (Pin_20), MX-Down1.1 (COL), MX-Hm1.1 (COL), MX-Up1.1 (COL), MX-end1.1 (COL)
- removed net Col16: J1.21 (Pin_21), MX-PgDn1.1 (COL), MX-PgUp1.1 (COL), MX-Right1.1 (COL)
- new net: MX-Up1.1 (COL), MX-end1.1 (COL)
Other:
- moved on the sheet: D15, D16, D17, D31, D32, D33, D59, D60, D64, D65, D66, D67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

Commit message: The Routing Continues
Connections:
- net Col12: now also MX-Up1.1 (COL), MX-end1.1 (COL)
Other:
- moved on the sheet: D1, D10, D11, D12, D13, D14, D15, D16, D17, D18, D19, D2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

Commit message: Version 0.1 Complete
Parts:
- J1: value Conn_01x18_Female -> Conn_01x20_Female; footprint Connector_PinHeader_2.54mm:PinHeader_1x18_P2.54mm_Vertical -> Connector_PinHeader_2.54mm:PinHeader_1x20_P2.54mm_Vertical; symbol Connector:Conn_01x18_Female -> Connector:Conn_01x20_Female
Connections:
- net Col0: now also J1.7 (Pin_7); no longer J1.5 (Pin_5)
- net Col1: now also J1.8 (Pin_8); no longer J1.6 (Pin_6)
- net Col10: now also J1.17 (Pin_17); no longer J1.15 (Pin_15)
- net Col11: now also J1.18 (Pin_18); no longer J1.16 (Pin_16)
- net Col12: now also J1.19 (Pin_19); no longer J1.17 (Pin_17)
- net Col13: now also J1.20 (Pin_20); no longer J1.18 (Pin_18)
- net Col2: now also J1.9 (Pin_9); no longer J1.7 (Pin_7)
- net Col3: now also J1.10 (Pin_10); no longer J1.8 (Pin_8)
- net Col4: now also J1.11 (Pin_11); no longer J1.9 (Pin_9)
- net Col5: now also J1.12 (Pin_12); no longer J1.10 (Pin_10)
- net Col6: now also J1.13 (Pin_13); no longer J1.11 (Pin_11)
- net Col7: now also J1.14 (Pin_14); no longer J1.12 (Pin_12)
- net Col8: now also J1.15 (Pin_15); no longer J1.13 (Pin_13)
- net Col9: now also J1.16 (Pin_16); no longer J1.14 (Pin_14)
- net Row3: now also J1.4 (Pin_4)
- net Row4: now also J1.5 (Pin_5); no longer J1.4 (Pin_4)
Changed lines of the file:
@@
 $EndDescr
 $Comp
-L Connector:Conn_01x18_Female J1
+L Connector:Conn_01x20_Female J1
 U 1 1 5FBC2DAD
 P 5650 1050
 F 0 "J1" V 5815 1030 50  0000 C CNN
-F 1 "Conn_01x18_Female" V 5724 1030 50  0000 C CNN
-F 2 "Connector_PinHeader_2.54mm:PinHeader_1x18_P2.54mm_Vertical" H 5650 1050 50  0001 C CNN
+F 1 "Conn_01x20_Female" V 5724 1030 50  0000 C CNN
+F 2 "Connector_PinHeader_2.54mm:PinHeader_1x20_P2.54mm_Vertical" H 5650 1050 50  0001 C CNN
 F 3 "~" H 5650 1050 50  0001 C CNN
 	1    5650 1050
@@
 Text GLabel 9450 2150 1    50   Input ~ 0
 Col13
-Text GLabel 5250 1250 3    50   Input ~ 0
+Text GLabel 5350 1250 3    50   Input ~ 0
 Col0
-Text GLabel 5350 1250 3    50   Input ~ 0
+Text GLabel 5450 1250 3    50   Input ~ 0
 Col1
-Text GLabel 5450 1250 3    50   Input ~ 0
+Text GLabel 5550 1250 3    50   Input ~ 0
 Col2
-Text GLabel 5550 1250 3    50   Input ~ 0
+Text GLabel 5650 1250 3    50   Input ~ 0
 Col3
-Text GLabel 5650 1250 3    50   Input ~ 0
+Text GLabel 5750 1250 3    50   Input ~ 0
 Col4
-Text GLabel 5750 1250 3    50   Input ~ 0
+Text GLabel 5850 1250 3    50   Input ~ 0
 Col5
-Text GLabel 5850 1250 3    50   Input ~ 0
+Text GLabel 5950 1250 3    50   Input ~ 0
 Col6
-Text GLabel 5950 1250 3    50   Input ~ 0
+Text GLabel 6050 1250 3    50   Input ~ 0
 Col7
-Text GLabel 6050 1250 3    50   Input ~ 0
+Text GLabel 6150 1250 3    50   Input ~ 0
 Col8
-Text GLabel 6150 1250 3    50   Input ~ 0
+Text GLabel 6250 1250 3    50   Input ~ 0
 Col9
-Text GLabel 6250 1250 3    50   Input ~ 0
+Text GLabel 6350 1250 3    50   Input ~ 0
 Col10
-Text GLabel 6350 1250 3    50   Input ~ 0
+Text GLabel 6450 1250 3    50   Input ~ 0
 Col11
-Text GLabel 6450 1250 3    50   Input ~ 0
+Text GLabel 6550 1250 3    50   Input ~ 0
 Col12
-Text GLabel 6550 1250 3    50   Input ~ 0
+Text GLabel 6650 1250 3    50   Input ~ 0
 Col13
+Text GLabel 4750 1250 3    50   Input ~ 0
+Row0
 Text GLabel 4850 1250 3    50   Input ~ 0
-Row0
+Row1
 Text GLabel 4950 1250 3    50   Input ~ 0
-Row1
-Text GLabel 5050 1250 3    50   Input ~ 0
 Row2
 Text GLabel 5150 1250 3    50   Input ~ 0
@@
 	8900 6050 8900 5150
 Connection ~ 8900 5150
+Text GLabel 5050 1250 3    50   Input ~ 0
+Row3
 $EndSCHEMATC
